File: hardware/pcb/unnamed-programmer.sch (EAGLE design)
At the start: 16 parts, among them U1 FT4232H-56Q

Commit message: sch work
Parts:
- added C13, C16, C17: 100n, Passive Components > Capacitors > Multilayer Ceramic Capacitors MLCC:MLCC0603
- added C14, C15: 27p, Passive Components > Capacitors > Multilayer Ceramic Capacitors MLCC:MLCC0603
- added D1: SP0503BAHT, Circuit Protection > ESD Suppressors \ TVS Diodes:SP0503BAHT
- added F1: (no value), Circuit Protection > Resettable Fuses - PPTC:PTC0805
- added J1: USB-C, Connectors > USB:USB-C
- added J2: 20, Connectors > Header:20
- added L3: (no value), Passive Components > Inductors, Chokes & Coils:INDUCTOR_6X6MM
- added R10, R11, R3, R5, R6: 10k, Passive Components > Resistors > Chip Resistors:RESISTOR0603
- added R2: 2k2, Passive Components > Resistors > Chip Resistors:RESISTOR0603
- added R4: 4k7, Passive Components > Resistors > Chip Resistors:RESISTOR0603
- added R7: 100k, Passive Components > Resistors > Chip Resistors:RESISTOR0603
- added R8, R9: xk, Passive Components > Resistors > Chip Resistors:RESISTOR0603
- added U2: MIC24045, Power > Switching Controllers:MIC24045
- added U3: 93LC46B, Semiconductors > Integrated Circuits - ICs > Memory ICs > EEPROM:93LC46B
- added U4, U5: 74LVC8T245, Semiconductors > Integrated Circuits - ICs > Logic ICs > Logic Gates:74LVC8T245
- added U6: 74LVC1G125, Semiconductors > Integrated Circuits - ICs > Logic ICs > Logic Gates:74LVC1G125
- added X1: 12MHz, Passive Components > Frequency Control & Timing Devices > Crystals:CRYSTAL_4P
- C1, C10, C11, C12, C2, C3, C4, C7: value 100nF -> 100n; device Capacitor:CAPACITOR-0603 -> Passive Components > Capacitors > Multilayer Ceramic Capacitors MLCC:MLCC0603
- C5: value 1uF -> 1u; device Capacitor:CAPACITOR-0603 -> Passive Components > Capacitors > Multilayer Ceramic Capacitors MLCC:MLCC0603
- C6: value 3.3uF -> 100n; device Capacitor:CAPACITOR-0603 -> Passive Components > Capacitors > Multilayer Ceramic Capacitors MLCC:MLCC0603
- C8, C9: value 4.7uF -> 4u7; device Capacitor:CAPACITOR-0603 -> Passive Components > Capacitors > Multilayer Ceramic Capacitors MLCC:MLCC0603
- L1, L2: value 350nH -> 350nH 1.4A; device Inductor:INDUCTOR-0603 -> Passive Components > Inductors, Chokes & Coils:INDUCTOR_NC_0603; CURRENT 1.4A -> (none); OCMOUSER 81-BLM18PG221SN1D -> (none)
- R1: value 12K Ohms -> 12k 1%; device Resistor:RESISTOR-0603 -> Passive Components > Resistors > Chip Resistors:RESISTOR0603; TOLERANCE 1% -> (none)
- U1: device FTDI:FT4232H-56Q -> Semiconductors > Integrated Circuits - ICs > Interface ICs > USB Interface IC:FT4232H-56Q
Connections:
- removed net 3V3: C1.C1, C2.C1, C3.C1, C4.C1, C5.C1, L1.1, L2.1, U1.VCCIO@0, U1.VCCIO@1, U1.VCCIO@2, U1.VREGIN
- removed net FT_EE_SCL: U1.EECLK
- removed net FT_EE_SDA: U1.EEDATA
- new net !OE: U5.!OE
- new net 3.3V: C1.P$1, C13.P$1, C16.P$1, C17.P$1, C2.P$1, C3.P$1, C4.P$1, C5.P$1, L1.P$2, L2.P$2, R3.P$2, R5.P$2, R6.P$2, U1.VCCIO@0, U1.VCCIO@1, U1.VCCIO@2, U1.VREGIN, U3.ORG, U3.VCC, U4.VCCA, U5.DIR, U5.VCCA, U6.PW.VCC
- new net 3.3V1: R10.P$2, R11.P$2
- new net 5V: D1.4, F1.1, J2.19.S, R4.P$2
- new net DBGRQ: J2.17.S
- new net FT_EE_CLK: R5.P$1, U1.EECLK, U3.CLK
- new net FT_EE_DAT: R2.P$1, U1.EEDATA, U3.DI
- new net FT_SCL: R11.P$1, U1.BDBUS0, U2.SCL
- new net FT_SDA: R10.P$1, U1.BDBUS1, U1.BDBUS2, U2.SDA
- new net N$10: J1.SBU2@B8, R8.P$2
- new net N$11: J1.SBU1@A8, R9.P$2
- new net N$5: R2.P$2, R3.P$1, U3.DO
- new net N$6: C15.P$1, U1.OSCO, X1.2
- new net N$7: R4.P$1, R7.P$2, U1.!RESET
- new net N$8: C14.P$1, U1.OSCI, X1.1
- new net N$9: F1.2, J1.VBUS@A4,A9,B9,B4
- new net NTRST: J2.3.S
- new net RESET: J2.15.S, U6.1.Y
- new net RESET_: U6.1.A
- new net REST_OE: U6.1.OE
- new net RTCK: J2.11.S
- new net SWCLK/TCK: J2.9.S
- new net SWDIO/TMS: J2.7.S
- new net SWO/TDO: J2.13.S
- new net TDI: J2.5.S
- new net VSUP: J2.2.S
- new net VTREF: J2.1.S, U4.VCCB, U5.VCCB
- net !FT_EE_CS: now also R6.P$1, U3.CS
- net GND: now also C1.P$2, C10.P$2, C11.P$2, C12.P$2, C13.P$2, C14.P$2, C15.P$2, C16.P$2, C17.P$2, C2.P$2, C3.P$2, C4.P$2, C5.P$2, C6.P$2, C7.P$2, C8.P$2, C9.P$2, D1.1, J1.GND@A1,A12,B12,B1, J1.SHIELD, J2.10.S, J2.12.S, J2.14.S, J2.16.S, J2.18.S, J2.20.S, J2.4.S, J2.6.S, J2.8.S, R1.P$1, R7.P$1, R8.P$1, R9.P$1, U2.AGND, U2.PGND@0, U2.PGND@1, U2.PGND@2, U2.PGND@3, U3.VSS, U4.!OE, U4.DIR, U4.GND, U5.GND, U6.PW.GND, X1.GND@0, X1.GND@1; no longer C1.C2, C10.C2, C11.C2, C12.C2, C2.C2, C3.C2, C4.C2, C5.C2, C6.C2, C7.C2, C8.C2, C9.C2, R1.1
- net N$1: now also R1.P$2; no longer R1.2
- net N$2: now also C11.P$1, C12.P$1, C6.P$1; no longer C11.C1, C12.C1, C6.C1
- net N$3: now also C10.P$1, C9.P$1, L2.P$1; no longer C10.C1, C9.C1, L2.2
- net N$4: now also C7.P$1, C8.P$1, L1.P$1; no longer C7.C1, C8.C1, L1.2
- net USB_DM: now also D1.3, J1.DN@A7,B7
- net USB_DP: now also D1.2, J1.DP@A6,B6
Other:
- note added: "***"
- note added: "COM port 1"
- note added: "COM port 2"
- note added: "Control interface"
- note added: "Inputs"
- note added: "JTAG interface connection (20 pin )J-Link and J-Trace have a JTAG connector compatible to ARM's Multi-ICE. The JTAG connector is a 20 way Insulation Displacement Connector (IDC) keyed box header(2.54mm male) that mates with IDC sockets mounted on a ribbon cable. *On later J-Link products like the J-Link ULTRA+, these pinsare reserved for firmware extension purposes. They can be left open or conne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"
- note added: "Outputs"
- note added: "Programing Interface"
- note added: "TEMPORARY"
- note added: "TODO: Mudar para TSSOP24, cuz espensive"
- note added: "TODO: Select inductor"
- moved on the sheet: U1
